Commit message: Add SimplerEnv-OpenVLA specific modifications
- Added Jaco robot support with configs and robot definition
- Enhanced base agent and controller functionality
- Updated custom environments for improved scene handling
- Added ADA robot description assets
- Modified various robot controllers for better compatibility
- Updated requirements and environment configurations

🤖 Generated with [Claude Code](https://claude.ai/code)

Co-Authored-By: Claude <noreply@anthropic.com>

File: data/custom/mk_station.urdf (robot description, URDF)
Before this commit: robot mk_station, 4 links, 3 joints
Links:
- removed link middle_drawer
- link body: geometry collision box size=0.01 0.3075 0.3075; collision box size=0.295 0.01 0.3075
- link bottom_drawer: geometry collision box size=0.0075 0.2875 0.14; collision box size=0.01 0.2575 0.05
- link top_drawer: geometry collision box size=0.0075 0.2875 0.14; collision box size=0.01 0.2575 0.05
Joints:
- removed joint middle_drawer_joint
- joint bottom_drawer_joint: limit lower=0 upper=0.5 effort=0.00000 velocity=0.00000 -> lower=0.0 upper=0.25 effort=0.00000 velocity=0.00000; origin xyz=0.00000 0.00000 0.17800 rpy=0.00000 0.00000 0.00000 -> xyz=0.0 0.0 0.064 rpy=0.00000 0.00000 0.00000
- joint top_drawer_joint: limit lower=0 upper=0.5 effort=0.00000 velocity=0.00000 -> lower=0.0 upper=0.25 effort=0.00000 velocity=0.00000; origin xyz=0.00000 0.00000 0.66800 rpy=0.00000 0.00000 0.00000 -> xyz=0.0 0.0 0.2165 rpy=0.00000 0.00000 0.00000
